File: nice_pillz.kicad_sch (KiCad schematic)
At the start: 20 parts, among them J1 Conn_01x13, J2 Conn_01x13, J3 Conn_01x13, J4 Conn_01x13, J5 Conn_01x10, J6 Conn_01x10, J7 Conn_01x13, J8 Conn_01x13, SW1 RESET, U1 nice!nano V2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

Commit message: full update
Parts:
- added J10: BatteryTerminal, TerminalBlock:TerminalBlock_Xinya_XY308-2.54-2P_1x02_P2.54mm_Horizontal, symbol Connector:Screw_Terminal_01x02
- added J9: ChassisButton, TerminalBlock:TerminalBlock_Xinya_XY308-2.54-2P_1x02_P2.54mm_Horizontal, symbol Connector:Screw_Terminal_01x02
Connections:
- net BAT+: now also J10.2 (Pin_2), J9.2 (Pin_2); no longer U1.24 (B0)
- new net BAT: J9.1 (Pin_1), U1.24 (B0)
- new net BAT-: J10.1 (Pin_1)
