File: nice_pillz.kicad_pcb (KiCad board)
At the start: 2 copper layers, 100 x 86 mm, 25 parts, among them J1 Conn_01x13, J2 Conn_01x13, J3 Conn_01x13, J4 Conn_01x13, J5 Conn_01x10, J6 Conn_01x10, J7 Conn_01x13, J8 Conn_01x13, M1 MountingHole_6.4mm_M6, M3 MountingHole_4.3mm_M4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

Commit message: full update
Parts:
- removed Batterie Connector: TerminalBlock_CUI_TB007-508-02_1x02_P5.08mm_Horizontal, TerminalBlock_CUI:TerminalBlock_CUI_TB007-508-02_1x02_P5.08mm_Horizontal
- removed Case Switch: TerminalBlock_CUI_TB007-508-02_1x02_P5.08mm_Horizontal, TerminalBlock_CUI:TerminalBlock_CUI_TB007-508-02_1x02_P5.08mm_Horizontal
- removed G***: LOGO, pillz:pillz_logo
- added Battery: TerminalBlock_Xinya_XY308-2.54-2P_1x02_P2.54mm_Horizontal, TerminalBlock:TerminalBlock_Xinya_XY308-2.54-2P_1x02_P2.54mm_Horizontal, B.Cu at (167.8, 128.1)
- added Chassis Switch: TerminalBlock_Xinya_XY308-2.54-2P_1x02_P2.54mm_Horizontal, TerminalBlock:TerminalBlock_Xinya_XY308-2.54-2P_1x02_P2.54mm_Horizontal, B.Cu at (172.9, 60.3)
Routing:
- net /ROW_13: track 252.1 -> 190.9 mm
- net /COL_4: track 206.2 -> 197.4 mm
- net /ROW_2: track 61.3 -> 58.2 mm
- net /ROW_3: track 76.5 -> 73.7 mm
- net /COL_3: track 203.9 -> 201.4 mm
- net /COL_2: track 200.7 -> 199.2 mm
- net /ROW_12: track 177.7 -> 176.4 mm
- net /COL_5: track 255.5 -> 256.8 mm
- net /COL_6: track 173.0 -> 171.9 mm
- net /SPI_MOSI: track 32.1 -> 31.0 mm
- net BAT: track 42.2 -> 43.2 mm
- net /COL_1: track 199.6 -> 198.7 mm
- net /COL_0: track 203.2 -> 202.3 mm
- net /ROW_4: track 84.9 -> 85.3 mm, vias 3 -> 2
- net /ROW_0: track 46.2 -> 46.5 mm, vias 1 -> 0
Other:
- board text added: "Nice Pillz github.com/nol00p/nicepillz v0.1"
- board text removed: "KB600"
- board text removed: "KEYPAD"
- board text removed: "Molex 39-53-2135"
- board text removed: "Nice Pillz github.com/nol00p/nicepillz"
- board text removed: "Pillz Mod Pro github.com/dcpedit/pillzmod by dcpedit (Rev 2)"

Commit message: update 3d
Parts:
- added G***: LOGO, Local:NicePillz, F.Cu at (170.9, 88.9)
- added G***: LOGO, Local:NicePillz, B.Cu at (170.9, 89.0)

Commit message: battery connection
Parts:
- added ?: , , F.Cu at (150.2, 83.6)
- added ?: , , F.Cu at (150.3, 83.4)
Routing:
- net BAT-: track 0.00 -> 43.5 mm
- net GND: track 0.00 -> 10.8 mm
- net BAT: track 43.2 -> 45.8 mm

Commit message: Production files created
Parts:
- removed SW1: RESET, Button_Switch_SMD:SW_SPST_SKQG_WithoutStem
- added REF**: SW_PUSH_6mm, Button_Switch_THT:SW_PUSH_6mm, B.Cu at (140.4, 55.7)
Routing:
- net /ROW_8: track 95.0 -> 111.2 mm
- net /RESET: track 29.8 -> 33.5 mm
- net /ROW_3: track 73.7 -> 76.3 mm
- net /ROW_1: track 32.4 -> 30.6 mm
- net /ROW_10: track 52.5 -> 53.9 mm
- net +5V: track 31.9 -> 33.2 mm
- net /ROW_11: track 64.5 -> 65.8 mm
- net /ROW_13: track 190.9 -> 189.8 mm
- net /COL_0: track 202.3 -> 203.4 mm
- net /COL_1: track 198.7 -> 197.6 mm
- net /ROW_5: track 68.5 -> 69.5 mm
- net /ROW_6: track 133.9 -> 134.8 mm
- net /ROW_9: track 91.0 -> 90.2 mm
- net /COL_2: track 199.2 -> 198.5 mm
- net /ROW_7: track 103.2 -> 103.8 mm
Other:
- board text added: "Nice Pillz github.com/nol00p/nicepillz v1.0 Feb 26"
- board text removed: "Nice Pillz github.com/nol00p/nicepillz v0.1"
