File: Board/nice_pillz.kicad_pcb (KiCad board)
At the start: 2 copper layers, 100 x 86 mm, 26 parts, among them J1 Conn_01x13, J2 Conn_01x13, J3 Conn_01x13, J4 Conn_01x13, J5 Conn_01x10, J6 Conn_01x10, J7 Conn_01x13, J8 Conn_01x13, M1 MountingHole_6.4mm_M6, M3 MountingHole_4.3mm_M4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

Commit message: clean up
Parts:
- added Ext. Reset Switch: TerminalBlock_Xinya_XY308-2.54-2P_1x02_P2.54mm_Horizontal, TerminalBlock:TerminalBlock_Xinya_XY308-2.54-2P_1x02_P2.54mm_Horizontal, B.Cu at (161.7, 60.2)
- Ext. PWR Switch: renamed from Chassis Switch
Routing:
- net /RESET: track 33.5 -> 58.0 mm
